File: Timagotchi.kicad_pcb (KiCad board)
At the start: 2 copper layers, 98 x 53.5 mm, 10 parts, among them J1 Conn_01x13_Pin, J2 Conn_01x02_Pin, SW1 SW_Omron_B3FS, SW2 SW_Omron_B3FS, SW3 SW_Omron_B3FS, SW4 SW_Omron_B3FS, SW5 SW_Omron_B3FS, SW6 SW_Omron_B3FS, U1 XIAO-ESP32-S3-Plus-SMD, U2 MAX98357A

Commit message: pcb joystick
Parts:
- added U3: COM-09032, Joystick footprint:XDCR_COM-09032, F.Cu at (82.5, 100.3)
- moved SW1 147.2 mm to (55.0, 51.2)
- moved SW2 147.2 mm to (55.0, 59.1)
- moved SW3 147.2 mm to (55.0, 67.0)
- moved SW4 147.2 mm to (55.0, 74.8)
- moved SW5 147.2 mm to (55.0, 82.7)
- moved SW6 147.2 mm to (55.0, 90.5)
- moved U1 55.7 mm to (94.0, 69.2)
- moved J1 39.8 mm to (118.0, 86.0)
- moved J2 15.8 mm to (143.8, 99.9), turned to 0 degrees
- moved U2 5.54 mm to (143.8, 106.4)
Connections:
- U1 pad 25: unconnected-(U1-GPIO40_MTDO_CAM_SDA_I2S_WS-Pad25) -> /SEL
- U1 pad 28: unconnected-(U1-GPIO42_MTMS_PDM_CLK_TX1-Pad28) -> /HPOS
- U1 pad 29: unconnected-(U1-GPIO39_MTCK_CAM_SCL_I2S_SCK-Pad29) -> /VPOS
Routing:
- net GND: track 14.4 -> 0.00 mm
- net /VBAT: track 9.79 -> 0.00 mm
- net /I2S_WS: track 5.92 -> 0.00 mm
- net /I2S_SCK: track 4.13 -> 0.00 mm
- net /I2S_SD: track 3.85 -> 0.00 mm
- net /MOSI: track 1.98 -> 0.00 mm, vias 1 -> 0
Other:
- board outline removed
