File: Timagotchi.kicad_sch (KiCad schematic)
At the start: 2 parts, among them J1 Conn_01x13_Pin, U1 XIAO-ESP32-S3-Plus-SMD

Commit message: got battery pins and screen setup :)
Parts:
- added J2: Conn_01x02_Pin, Connector_JST:JST_PH_B2B-PH-K_1x02_P2.00mm_Vertical, symbol Connector:Conn_01x02_Pin
Connections:
- net VCC: now reaches J1.1 (Pin_1)
- net VCC: now also U1.12 (3V3)
- net TP_SDA: now reaches J1.10 (Pin_10)
- net TP_SDA: now also U1.5 (GPIO5_A4_D4_SDA)
- net TP_SCL: now reaches J1.11 (Pin_11)
- net TP_SCL: now also U1.6 (GPIO6_A5_D5_SCL)
- net TP_INT: now reaches J1.12 (Pin_12)
- net TP_INT: now also U1.1 (GPIO1_A0_D0)
- net TP_RST: now reaches J1.13 (Pin_13)
- net TP_RST: now also U1.10 (GPIO8_A9_D9_MISO)
- net GND: now reaches J1.2 (Pin_2)
- net GND: now also U1.13 (GND)
- net MOSI: now reaches J1.3 (Pin_3)
- net MOSI: now also U1.11 (GPIO9_A10_D10_MOSI)
- net SCLK: now reaches J1.4 (Pin_4)
- net SCLK: now also U1.9 (GPIO7_A8_D8_SCK)
- net SD_CS: now reaches J1.5 (Pin_5)
- net SD_CS: now also U1.2 (GPIO2_A1_D1)
- net LCD_CS: now reaches J1.6 (Pin_6)
- net LCD_CS: now also U1.8 (GPIO44_D7_RX)
- net LCD_DC: now reaches J1.7 (Pin_7)
- net LCD_DC: now also U1.7 (GPIO43_D6_TX)
- net LCD_RST: now reaches J1.8 (Pin_8)
- net LCD_RST: now also U1.4 (GPIO4_A3_D3)
- net LCD_BL: now reaches J1.9 (Pin_9)
- net LCD_BL: now also U1.3 (GPIO3_A2_D2)

Commit message: something
Parts:
- added SW1, SW2, SW3, SW4, SW5, SW6: SW_Omron_B3FS, symbol Switch:SW_Omron_B3FS
- added U2: MAX98357A, Package_DFN_QFN:TQFN-16-1EP_3x3mm_P0.5mm_EP1.23x1.23mm, symbol Audio:MAX98357A
- U1: footprint Seeed_Studio_XIAO_Series:XIAO-ESP32-S3-Plus-SMD -> New_XIAO_Series_Footprints:XIAO-ESP32-S3-Plus-SMD
Connections:
- net GND: now also J2.2 (Pin_2), U1.33 (GND2), U1.34 (PAD), SW1.2, SW2.2, SW3.2, SW4.2, SW5.2, SW6.2, U2.11 (GND), U2.15 (GND), U2.17 (PAD), U2.3 (GND)
- net I2S_SD: now reaches U1.15 (GPIO38_DVP_VSYNC_I2S_SD)
- net I2S_SD: now also U2.1 (DIN)
- net I2S_SCK: now reaches U1.16 (GPIO39_CAM_SCL_I2S_SCK)
- net I2S_SCK: now also U2.16 (BCLK)
- net I2S_WS: now reaches U1.17 (GPIO40_CAM_SDA_I2S_WS)
- net I2S_WS: now also U2.14 (LRCLK)
- net SW4: now reaches U1.18 (GPIO41_PDM_DATA_RX1)
- net SW4: now also SW4.1
- net SW5: now reaches U1.19 (GPIO42_PDM_CLK_TX1)
- net SW5: now also SW5.1
- net SW6: now reaches U1.20 (GPIO10_XMCLK_ADC_BAT)
- net SW6: now also SW6.1
- net SW1: now reaches U1.21 (GPIO11_DVP_Y8_SPI_MOSI1)
- net SW1: now also SW1.1
- net SW2: now reaches U1.22 (GPIO12_DVP_Y7_SPI_MISO1)
- net SW2: now also SW2.1
- net SW3: now reaches U1.23 (GPIO13_DVP_PCLK_SPI_SCK1)
- net SW3: now also SW3.1
- net VBAT: now reaches U1.32 (VBAT)
- net VBAT: now also J2.1 (Pin_1)
- net VCC renamed +3.3V
- net +3.3V: now also U2.4 (~{SD_MODE}), U2.7 (VDD), U2.8 (VDD)
- no-connect marks 0 -> 3
Other:
- note added: "Battery"
- note added: "Buttons"
- note added: "Speaker"

Commit message: a bunch of stuff
Parts:
- SW1, SW2, SW3, SW4, SW5, SW6: footprint (none) -> Button_Switch_SMD:SW_SPST_Omron_B3FS-100xP
Connections:
- no-connect marks 3 -> 11
Changed lines of the file:
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@@
+	)
+	(no_connect
+		(at 90.17 80.01)
+	)
+	(no_connect
+		(at 90.17 90.17)
+	)
+	(no_connect
+		(at 90.17 72.39)
+	)
+	(no_connect
+		(at 90.17 77.47)
 	)
 	(no_connect
@@
 	)
 	(no_connect
+		(at 90.17 85.09)
+	)
+	(no_connect
+		(at 90.17 82.55)
+	)
+	(no_connect
 		(at 190.5 67.31)
+	)
+	(no_connect
+		(at 90.17 87.63)
+	)
+	(no_connect
+		(at 90.17 74.93)
 	)
 	(wire
@@
 			)
 		)
-		(property "Footprint" ""
+		(property "Footprint" "Button_Switch_SMD:SW_SPST_Omron_B3FS-100xP"
 			(at 151.13 102.87 0)
 			(hide yes)
@@
 			)
 		)
-		(property "Footprint" ""
+		(property "Footprint" "Button_Switch_SMD:SW_SPST_Omron_B3FS-100xP"
 			(at 115.57 116.84 0)
 			(hide yes)
@@
 			)
 		)
-		(property "Footprint" ""
+		(property "Footprint" "Button_Switch_SMD:SW_SPST_Omron_B3FS-100xP"
 			(at 151.13 116.84 0)
 			(hide yes)
@@
 			)
 		)
-		(property "Footprint" ""
+		(property "Footprint" "Button_Switch_SMD:SW_SPST_Omron_B3FS-100xP"
 			(at 133.35 102.87 0)
 			(hide yes)
@@
 			)
 		)
-		(property "Footprint" ""
+		(property "Footprint" "Button_Switch_SMD:SW_SPST_Omron_B3FS-100xP"
 			(at 115.57 102.87 0)
 			(hide yes)
@@
 			)
 		)
-		(property "Footprint" ""
+		(property "Footprint" "Button_Switch_SMD:SW_SPST_Omron_B3FS-100xP"
 			(at 133.35 116.84 0)
 			(hide yes)

Commit message: pcb joystick
Parts:
- added U3: COM-09032, Joystick footprint:XDCR_COM-09032, symbol COM-09032:COM-09032
Connections:
- net +3.3V: now also U3.B1A (SEL+), U3.H2 (H), U3.V2 (V)
- net GND: now also U3.H3 (H-), U3.S1 (SHIELD), U3.S2 (SHIELD), U3.S3 (SHIELD), U3.S4 (SHIELD), U3.V3 (V-)
- net SEL: now reaches U1.25 (GPIO40_MTDO_CAM_SDA_I2S_WS)
- net SEL: now also U3.B2A (SEL-)
- net HPOS: now reaches U1.28 (GPIO42_MTMS_PDM_CLK_TX1)
- net HPOS: now also U3.H1 (H+)
- net VPOS: now reaches U1.29 (GPIO39_MTCK_CAM_SCL_I2S_SCK)
- net VPOS: now also U3.V1 (V+)
- no-connect marks 11 -> 7
Other:
- note added: "Joystick"
