File: PCB/Timagotchi.kicad_pcb (KiCad board)
At the start: 2 copper layers, 75 x 27 mm, 9 parts, among them J1 Conn_01x04, J2 Conn_01x02_Pin, SW1 SW_Omron_B3FS, SW2 SW_Omron_B3FS, SW3 SW_Omron_B3FS, U1 XIAO-ESP32-S3-Plus-SMD, U2 MAX98357A

Commit message: new pcb bc the screen wont fit :( but its fixed.
Parts:
- added REF**: MountingHole_2.2mm_M2, MountingHole:MountingHole_2.2mm_M2, F.Cu at (211.0, 65.5)
- added REF**: MountingHole_2.2mm_M2, MountingHole:MountingHole_2.2mm_M2, F.Cu at (132.0, 65.5)
- added REF**: MountingHole_2.2mm_M2, MountingHole:MountingHole_2.2mm_M2, F.Cu at (132.0, 41.0)
- moved J1 9.12 mm to (143.0, 52.0)
Routing:
- net (no net): track 0.00 -> 10.9 mm
- net /HPOS: track 16.0 -> 25.6 mm
- net /VPOS: track 17.5 -> 25.9 mm
- net GND: track 94.5 -> 93.5 mm
Other:
- board size 75 x 27 mm -> 85 x 30 mm
